File: KiCad/WS2815_D1Mini.kicad_pcb (KiCad board)
At the start: 2 copper layers, 61 x 39.4 mm, 14 parts, among them J1 Conn_01x08_Female, J13 691411410004, J14 691411410004, J2 Conn_01x08_Female, U1 WeMos_D1_mini, U2 L7805

Commit message: Add 2 mounting holes + move 12V and GND in power
Parts:
- added H1: MountingHole_Pad, MountingHole:MountingHole_4.3mm_M4_DIN965_Pad, F.Cu at (157.8, 89.2)
- added H3: MountingHole_Pad, MountingHole:MountingHole_4.3mm_M4_DIN965_Pad, F.Cu at (114.8, 82.0)
- moved LOGO1 12.0 mm to (146.2, 88.5)
- moved LOGO2 10.5 mm to (145.3, 85.1)
Connections:
- J13 pad 1: +12V -> GNDPWR
- J13 pad 2: +12V -> GNDPWR
- J13 pad 3: GNDPWR -> +12V
- J13 pad 4: GNDPWR -> +12V
Routing:
- net +12V: track 75.1 -> 64.3 mm, vias 3 -> 2
- net GNDPWR: track 94.0 -> 97.4 mm, vias 5 -> 6
- net GND: track 35.3 -> 37.0 mm
- net /GPo_WS281x: track 23.7 -> 22.5 mm
Other:
- board text added: "12V×2|GND×2"
- board text added: "WS2815_D1Mini V1r1 (2022/09/04)"
- board text removed: "GND×2|12V×2"
- board text removed: "WS2815_D1Mini V1r0 (2022/08/28)"

Commit message: Add zip, bom and pos for jlc
Parts:
- added U3: L78M05CDT-TR, Package_TO_SOT_SMD:TO-252-2, F.Cu at (150.6, 74.4)
- C4: value 1u -> 10u; footprint Capacitor_SMD:C_0603_1608Metric -> Capacitor_SMD:C_1206_3216Metric
- moved C4 0.74 mm to (129.8, 78.5)
Routing:
- net GND: track 37.0 -> 40.7 mm
- net GNDPWR: track 97.4 -> 94.7 mm
- net +5V: track 22.5 -> 24.8 mm
- net +12V: track 64.3 -> 65.4 mm
