File: KiCad/WS2815_D1Mini.kicad_sch (KiCad schematic)
At the start: 14 parts, among them J1 Conn_01x08_Female, J13 691411410004, J14 691411410004, J2 Conn_01x08_Female, U1 WeMos_D1_mini

Commit message: Add 2 mounting holes + move 12V and GND in power
Parts:
- added H1, H3: (no value), symbol Mechanical:MountingHole_Pad
- J1, J2: footprint (none) -> Connector_PinHeader_2.54mm:PinHeader_1x08_P2.54mm_Vertical
- LOGO1: value (none) -> Logo_Open_Hardware_Large; footprint (none) -> GoInK:GoInK600
- LOGO2: value (none) -> Logo_Open_Hardware_Large; footprint (none) -> GoInK:GoInK400
- U2: value (none) -> L7805; footprint (none) -> Package_TO_SOT_THT:TO-220-3_Horizontal_TabDown
Connections:
- net +12V: now also J13.3 (Pin_3), J13.4 (Pin_4); no longer J13.1 (Pin_1), J13.2 (Pin_2)
- net GNDPWR: now also J13.1 (Pin_1), J13.2 (Pin_2); no longer J13.3 (Pin_3), J13.4 (Pin_4)
- no-connect marks 0 -> 2
Changed lines of the file:
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@@
   (junction (at 64.77 109.22) (diameter 0) (color 0 0 0 0)
   )
+  (no_connect (at 194.31 147.32))
+  (no_connect (at 194.31 156.21))
   (wire (pts (xy 109.22 113.03) (xy 110.49 113.03))
     (stroke (width 0) (type default) (color 0 0 0 0))
@@
   (label "GP_D6" (at 76.2 68.58 0)
     (effects (font (size 1.27 1.27)) (justify left bottom))
+  )
+  (symbol (lib_id "Mechanical:MountingHole_Pad") (at 194.31 153.67 0) (unit 1)
+    (in_bom yes) (on_board yes) (fields_autoplaced)
+    (property "Reference" "H3" (id 0) (at 196.85 151.1299 0)
+      (effects (font (size 1.27 1.27)) (justify left))
+    )
+    (property "Value" "" (id 1) (at 196.85 153.6699 0)
+      (effects (font (size 1.27 1.27)) (justify left))
+    )
+    (property "Footprint" "" (id 2) (at 194.31 153.67 0)
+      (effects (font (size 1.27 1.27)) hide)
+    )
+    (property "Datasheet" "~" (id 3) (at 194.31 153.67 0)
+      (effects (font (size 1.27 1.27)) hide)
+    )
+    (pin "1")
   )
   (symbol (lib_id "MCU_Module:WeMos_D1_mini") (at 66.04 63.5 0) (unit 1)
@@
     (in_bom yes) (on_board yes)
     (property "Reference" "U2" (id 0) (at 72.39 103.0732 0))
-    (property "Value" "" (id 1) (at 72.39 105.3846 0))
-    (property "Footprint" "" (id 2) (at 73.025 113.03 0)
+    (property "Value" "L7805" (id 1) (at 72.39 105.3846 0))
+    (property "Footprint" "Package_TO_SOT_THT:TO-220-3_Horizontal_TabDown" (id 2) (at 73.025 113.03 0)
       (effects (font (size 1.27 1.27) italic) (justify left) hide)
     )
@@
       (effects (font (size 1.27 1.27)) hide)
     )
-    (property "Value" "" (id 1) (at 242.57 143.51 0)
-      (effects (font (size 1.27 1.27)) hide)
-    )
-    (property "Footprint" "" (id 2) (at 242.57 133.35 0)
+    (property "Value" "Logo_Open_Hardware_Large" (id 1) (at 242.57 143.51 0)
+      (effects (font (size 1.27 1.27)) hide)
+    )
+    (property "Footprint" "GoInK:GoInK600" (id 2) (at 242.57 133.35 0)
       (effects (font (size 1.27 1.27)) hide)
     )
@@
       (effects (font (size 1.27 1.27)) (justify left))
     )
-    (property "Footprint" "" (id 2) (at 190.5 52.07 0)
+    (property "Footprint" "Connector_PinHeader_2.54mm:PinHeader_1x08_P2.54mm_Vertical" (id 2) (at 190.5 52.07 0)
       (effects (font (size 1.27 1.27)) hide)
     )
@@
     (pin "1")
   )
+  (symbol (lib_id "Mechanical:MountingHole_Pad") (at 194.31 144.78 0) (unit 1)
+    (in_bom yes) (on_board yes) (fields_autoplaced)
+    (property "Reference" "H1" (id 0) (at 196.85 142.2399 0)
+      (effects (font (size 1.27 1.27)) (justify left))
+    )
+    (property "Value" "" (id 1) (at 196.85 144.7799 0)
+      (effects (font (size 1.27 1.27)) (justify left))
+    )
+    (property "Footprint" "" (id 2) (at 194.31 144.78 0)
+      (effects (font (size 1.27 1.27)) hide)
+    )
+    (property "Datasheet" "~" (id 3) (at 194.31 144.78 0)
+      (effects (font (size 1.27 1.27)) hide)
+    )
+    (pin "1")
+  )
   (symbol (lib_id "power:GND") (at 177.8 109.22 0) (unit 1)
     (in_bom yes) (on_board yes)
@@
     (pin "1")
   )
-  (symbol (lib_id "Connector:Conn_01x04_Female") (at 138.43 31.75 0) (unit 1)
-    (in_bom yes) (on_board yes)
-    (property "Reference" "J13" (id 0) (at 139.1412 31.2166 0)
-      (effects (font (size 1.27 1.27)) (justify left))
-    )
-    (property "Value" "691411410004" (id 1) (at 139.1412 33.528 0)
-      (effects (font (size 1.27 1.27)) (justify left))
-    )
-    (property "Footprint" "Wurth:WR-TBL-7.62mm-4P_691411410004" (id 2) (at 138.43 31.75 0)
-      (effects (font (size 1.27 1.27)) hide)
-    )
-    (property "Datasheet" "~" (id 3) (at 138.43 31.75 0)
-      (effects (font (size 1.27 1.27)) hide)
-    )
-    (property "Info" "Power" (id 4) (at 139.1412 35.8394 0)
+  (symbol (lib_id "Connector:Conn_01x04_Female") (at 138.43 34.29 0) (mirror x) (unit 1)
+    (in_bom yes) (on_board yes)
+    (property "Reference" "J13" (id 0) (at 139.1412 34.8234 0)
+      (effects (font (size 1.27 1.27)) (justify left))
+    )
+    (property "Value" "691411410004" (id 1) (at 139.1412 32.512 0)
+      (effects (font (size 1.27 1.27)) (justify left))
+    )
+    (property "Footprint" "Wurth:WR-TBL-7.62mm-4P_691411410004" (id 2) (at 138.43 34.29 0)
+      (effects (font (size 1.27 1.27)) hide)
+    )
+    (property "Datasheet" "~" (id 3) (at 138.43 34.29 0)
+      (effects (font (size 1.27 1.27)) hide)
+    )
+    (property "Info" "Power" (id 4) (at 139.1412 30.2006 0)
       (effects (font (size 1.27 1.27)) (justify left))
     )
@@
       (effects (font (size 1.27 1.27)) hide)
     )
-    (property "Value" "" (id 1) (at 256.54 143.51 0)
-      (effects (font (size 1.27 1.27)) hide)
-    )
-    (property "Footprint" "" (id 2) (at 256.54 133.35 0)
+    (property "Value" "Logo_Open_Hardware_Large" (id 1) (at 256.54 143.51 0)
+      (effects (font (size 1.27 1.27)) hide)
+    )
+    (property "Footprint" "GoInK:GoInK400" (id 2) (at 256.54 133.35 0)
       (effects (font (size 1.27 1.27)) hide)
     )
@@
     (property "Reference" "J2" (id 0) (at 213.995 39.37 0))
     (property "Value" "Conn_01x08_Female" (id 1) (at 210.82 53.34 90))
-    (property "Footprint" "" (id 2) (at 213.36 54.61 0)
+    (property "Footprint" "Connector_PinHeader_2.54mm:PinHeader_1x08_P2.54mm_Vertical" (id 2) (at 213.36 54.61 0)
       (effects (font (size 1.27 1.27)) hide)
     )
@@
       (reference "C4") (unit 1) (value "1u") (footprint "Capacitor_SMD:C_0603_1608Metric")
     )
+    (path "/57e17378-f1f7-42d0-9ad3-fb44c2d5cdc3"
+      (reference "H1") (unit 1) (value "MountingHole_Pad") (footprint "MountingHole:MountingHole_4.3mm_M4_DIN965_Pad")
+    )
+    (path "/01c950c2-84d4-4062-97ce-28407e323c63"
+      (reference "H3") (unit 1) (value "MountingHole_Pad") (footprint "MountingHole:MountingHole_4.3mm_M4_DIN965_Pad")
+    )
     (path "/250e8ef0-cb88-431e-905b-cd099b6598bf"

Commit message: Add zip, bom and pos for jlc
Parts:
- added U3: L78M05CDT-TR, Package_TO_SOT_SMD:TO-252-2, symbol Regulator_Linear:L7805
- C4: value 1u -> 10u; footprint Capacitor_SMD:C_0603_1608Metric -> Capacitor_SMD:C_1206_3216Metric; Umax (none) -> 16V
- H1, H3: value (none) -> MountingHole_Pad; footprint (none) -> MountingHole:MountingHole_4.3mm_M4_DIN965_Pad
Connections:
- net +12V: now also U3.1 (IN)
- net +5V: now also U3.3 (OUT)
- net GNDPWR: now also U3.2 (GND)
Changed lines of the file:
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@@
+    (stroke (width 0) (type default) (color 0 0 0 0))
+  )
+  (wire (pts (xy 82.55 133.35) (xy 80.01 133.35))
     (stroke (width 0) (type default) (color 0 0 0 0))
   )
@@
   )
   (wire (pts (xy 88.9 63.5) (xy 76.2 63.5))
+    (stroke (width 0) (type default) (color 0 0 0 0))
+  )
+  (wire (pts (xy 62.23 133.35) (xy 64.77 133.35))
     (stroke (width 0) (type default) (color 0 0 0 0))
   )
@@
       (effects (font (size 1.27 1.27)) (justify left))
     )
-    (property "Value" "" (id 1) (at 196.85 153.6699 0)
-      (effects (font (size 1.27 1.27)) (justify left))
-    )
-    (property "Footprint" "" (id 2) (at 194.31 153.67 0)
+    (property "Value" "MountingHole_Pad" (id 1) (at 196.85 153.6699 0)
+      (effects (font (size 1.27 1.27)) (justify left))
+    )
+    (property "Footprint" "MountingHole:MountingHole_4.3mm_M4_DIN965_Pad" (id 2) (at 194.31 153.67 0)
       (effects (font (size 1.27 1.27)) hide)
     )
     (property "Datasheet" "~" (id 3) (at 194.31 153.67 0)
+      (effects (font (size 1.27 1.27)) hide)
+    )
+    (pin "1")
+  )
+  (symbol (lib_id "power:GNDPWR") (at 72.39 140.97 0) (unit 1)
+    (in_bom yes) (on_board yes)
+    (property "Reference" "#PWR0122" (id 0) (at 72.39 146.05 0)
+      (effects (font (size 1.27 1.27)) hide)
+    )
+    (property "Value" "GNDPWR" (id 1) (at 72.4916 144.8816 0))
+    (property "Footprint" "" (id 2) (at 72.39 142.24 0)
+      (effects (font (size 1.27 1.27)) hide)
+    )
+    (property "Datasheet" "" (id 3) (at 72.39 142.24 0)
       (effects (font (size 1.27 1.27)) hide)
     )
@@
     (pin "8")
   )
+  (symbol (lib_id "power:+12V") (at 62.23 133.35 0) (unit 1)
+    (in_bom yes) (on_board yes)
+    (property "Reference" "#PWR0124" (id 0) (at 62.23 137.16 0)
+      (effects (font (size 1.27 1.27)) hide)
+    )
+    (property "Value" "+12V" (id 1) (at 62.611 128.9558 0))
+    (property "Footprint" "" (id 2) (at 62.23 133.35 0)
+      (effects (font (size 1.27 1.27)) hide)
+    )
+    (property "Datasheet" "" (id 3) (at 62.23 133.35 0)
+      (effects (font (size 1.27 1.27)) hide)
+    )
+    (pin "1")
+  )
   (symbol (lib_id "power:PWR_FLAG") (at 167.64 109.22 0) (unit 1)
     (in_bom yes) (on_board yes)
@@
       (effects (font (size 1.27 1.27)) (justify left))
     )
-    (property "Value" "" (id 1) (at 196.85 144.7799 0)
-      (effects (font (size 1.27 1.27)) (justify left))
-    )
-    (property "Footprint" "" (id 2) (at 194.31 144.78 0)
+    (property "Value" "MountingHole_Pad" (id 1) (at 196.85 144.7799 0)
+      (effects (font (size 1.27 1.27)) (justify left))
+    )
+    (property "Footprint" "MountingHole:MountingHole_4.3mm_M4_DIN965_Pad" (id 2) (at 194.31 144.78 0)
       (effects (font (size 1.27 1.27)) hide)
     )
@@
     (pin "1")
   )
+  (symbol (lib_id "Regulator_Linear:L7805") (at 72.39 133.35 0) (unit 1)
+    (in_bom yes) (on_board yes)
+    (property "Reference" "U3" (id 0) (at 72.39 127.2032 0))
+    (property "Value" "L78M05CDT-TR" (id 1) (at 72.39 129.5146 0))
+    (property "Footprint" "Package_TO_SOT_SMD:TO-252-2" (id 2) (at 73.025 137.16 0)
+      (effects (font (size 1.27 1.27) italic) (justify left) hide)
+    )
+    (property "Datasheet" "http://www.st.com/content/ccc/resource/technical/document/datasheet/41/4f/b3/b0/12/d4/47/88/CD00000444.pdf/files/CD00000444.pdf/jcr:content/translations/en.CD00000444.pdf" (id 3) (at 72.39 134.62 0)
+      (effects (font (size 1.27 1.27)) hide)
+    )
+    (property "LCSC" "C55509" (id 4) (at 72.39 133.35 0)
+      (effects (font (size 1.27 1.27)) hide)
+    )
+    (pin "1")
+    (pin "2")
+    (pin "3")
+  )
   (symbol (lib_id "Connector:Conn_01x04_Female") (at 138.43 34.29 0) (mirror x) (unit 1)
     (in_bom yes) (on_board yes)
@@
     )
     (pin "1")
-  )
-  (symbol (lib_id "Device:C") (at 86.36 33.02 0) (unit 1)
-    (in_bom yes) (on_board yes)
-    (property "Reference" "C4" (id 0) (at 89.281 31.8516 0)
-      (effects (font (size 1.27 1.27)) (justify left))
-    )
-    (property "Value" "1u" (id 1) (at 89.281 34.163 0)
-      (effects (font (size 1.27 1.27)) (justify left))
-    )
-    (property "Footprint" "Capacitor_SMD:C_0603_1608Metric" (id 2) (at 87.3252 36.83 0)
-      (effects (font (size 1.27 1.27)) hide)
-    )
-    (property "Datasheet" "~" (id 3) (at 86.36 33.02 0)
-      (effects (font (size 1.27 1.27)) hide)
-    )
-    (pin "1")
-    (pin "2")
   )
   (symbol (lib_id "Connector:Conn_01x08_Female") (at 213.36 54.61 180) (unit 1)
@@
     (pin "8")
   )
+  (symbol (lib_id "Device:C") (at 86.36 33.02 0) (unit 1)
+    (in_bom yes) (on_board yes)
+    (property "Reference" "C4" (id 0) (at 89.281 31.8516 0)
+      (effects (font (size 1.27 1.27)) (justify left))
+    )
+    (property "Value" "10u" (id 1) (at 89.281 34.163 0)
+      (effects (font (size 1.27 1.27)) (justify left))
+    )
+    (property "Footprint" "Capacitor_SMD:C_1206_3216Metric" (id 2) (at 87.3252 36.83 0)
+      (effects (font (size 1.27 1.27)) hide)
+    )
+    (property "Datasheet" "https://www.mouser.fr/ProductDetail/TDK/C3216X5R1C106M160AA" (id 3) (at 86.36 33.02 0)
+      (effects (font (size 1.27 1.27)) hide)
+    )
+    (property "Umax" "16V" (id 4) (at 86.36 33.02 0)
+      (effects (font (size 1.27 1.27)) hide)
+    )
+    (pin "1")
+    (pin "2")
+  )
+  (symbol (lib_id "power:+5V") (at 82.55 133.35 0) (unit 1)
+    (in_bom yes) (on_board yes)
+    (property "Reference" "#PWR0123" (id 0) (at 82.55 137.16 0)
+      (effects (font (size 1.27 1.27)) hide)
+    )
+    (property "Value" "+5V" (id 1) (at 82.931 128.9558 0))
+    (property "Footprint" "" (id 2) (at 82.55 133.35 0)
+      (effects (font (size 1.27 1.27)) hide)
+    )
+    (property "Datasheet" "" (id 3) (at 82.55 133.35 0)
+      (effects (font (size 1.27 1.27)) hide)
+    )
+    (pin "1")
+  )
   (symbol (lib_id "Connector:Conn_01x04_Female") (at 140.97 64.77 0) (unit 1)
     (in_bom yes) (on_board yes)
@@
       (reference "#PWR0121") (unit 1) (value "+5V") (footprint "")
     )
+    (path "/0e49aa81-d18a-4b07-a30e-e332fa277fd6"
+      (reference "#PWR0122") (unit 1) (value "GNDPWR") (footprint "")
+    )
+    (path "/dc30c6f2-6ff2-4f91-99ab-2bfa4259f28c"
+      (reference "#PWR0123") (unit 1) (value "+5V") (footprint "")
+    )
+    (path "/279960b8-b1ca-4d00-85fc-033958d91f97"
+      (reference "#PWR0124") (unit 1) (value "+12V") (footprint "")
+    )
     (path "/80fe070c-5552-4d5b-9daf-e06941e95f16"
       (reference "C1") (unit 1) (value "47u") (footprint "Capacitor_THT:CP_Radial_D5.0mm_P2.00mm")
@@
       (reference "C3") (unit 1) (value "10u") (footprint "Capacitor_SMD:C_1206_3216Metric")
     )
-    (path "/d2b287bc-2f46-4c35-bfa6-97b6a4a32736"
-      (reference "C4") (unit 1) (value "1u") (footprint "Capacitor_SMD:C_0603_1608Metric")
+    (path "/d91b978f-8137-4df8-8288-3fd62f8dd07e"
+      (reference "C4") (unit 1) (value "10u") (footprint "Capacitor_SMD:C_1206_3216Metric")
     )
     (path "/57e17378-f1f7-42d0-9ad3-fb44c2d5cdc3"
@@
       (reference "U2") (unit 1) (value "L7805") (footprint "Package_TO_SOT_THT:TO-220-3_Horizontal_TabDown")
     )
-  )
+    (path "/6fff55eb-076f-4a2f-86d3-091fcb2366e9"
+      (reference "U3") (unit 1) (value "L78M05CDT-TR") (footprint "Package_TO_SOT_SMD:TO-252-2")
+    )
+  )
